File: RFpuck_pro/RFpuck_pro.kicad_sch (KiCad schematic)
At the start: 1 part, among them U1 NRF24L01

Commit message: Tried to create a rf recever
Parts:
- removed U1: NRF24L01, Package_DFN_QFN:QFN-20-1EP_4x4mm_P0.5mm_EP2.5x2.5mm, symbol RF:NRF24L01
- added TP1: 5v, symbol Connector:TestPoint
- added TP2: GND, symbol Connector:TestPoint
- added U1: ESP32-C3, Package_DFN_QFN:QFN-32-1EP_5x5mm_P0.5mm_EP3.7x3.7mm, symbol MCU_Espressif:ESP32-C3
- added U2: SX1280IMLTRT, SX1280IMLTRT:XCVR_SX1280IMLTRT, symbol SX1280IMLTRT:SX1280IMLTRT
Connections:
- new net: U1.2 (VDD3P3), U1.3 (VDD3P3)
- new net: U1.31 (VDDA), U1.32 (VDDA)
- new net GND: TP2.1, U1.33 (GND), U2.13 (GND), U2.20 (GND), U2.21 (GND), U2.23 (GND), U2.24 (GND), U2.5 (GND)
