File: barrel-roll-nopcb/Untitled/Untitled.kicad_sch (KiCad schematic)
At the start: 12 parts, among them M1 Drive_Motor_DC, M2 Drive_Motor_DC, U2 DRV8833PW, U3 WeaponMotor, U4 Recever

Commit message: Tried to create a rf recever
Parts:
- removed U4: Recever, Connector_PinHeader_2.54mm:PinHeader_1x04_P2.54mm_Vertical, symbol New_Library:RP1_V2_ExpressLRS_2.4ghz_Nano_Receiver
