File: barrel-roll-DIPPCB/barrel-roll-DIPPCB_pro.kicad_sch (KiCad schematic)
At the start: 11 parts, among them M1 Motor_DC, M2 Motor_DC, U1 XIAO-RP2040-DIP, U2 DRV8833PW, U3 WeaponMotor, U4 Recever

Commit message: Updated PCB to have a DIP version and improved readme.
Parts:
- U1: footprint Seeed Studio XIAO Series Library:XIAO-RP2040-SMD -> Seeed Studio XIAO Series Library:XIAO-RP2040-DIP
Changed lines of the file:
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@@
 		)
 		(instances
-			(project "barrel-roll"
+			(project "barrel-roll-DIPPCB_pro"
 				(path "/78e1f998-c6c8-4383-a798-619907ba92a3"
 					(reference "U4")
@@
 		)
 		(instances
-			(project "barrel-roll"
+			(project "barrel-roll-DIPPCB_pro"
 				(path "/78e1f998-c6c8-4383-a798-619907ba92a3"
 					(reference "MX-5A_ESC1")
@@
 		)
 		(instances
-			(project "barrel-roll"
+			(project "barrel-roll-DIPPCB_pro"
 				(path "/78e1f998-c6c8-4383-a798-619907ba92a3"
 					(reference "TP5")
@@
 		)
 		(instances
-			(project "barrel-roll"
+			(project "barrel-roll-DIPPCB_pro"
 				(path "/78e1f998-c6c8-4383-a798-619907ba92a3"
 					(reference "M2")
@@
 		)
 		(instances
-			(project "barrel-roll"
+			(project "barrel-roll-DIPPCB_pro"
 				(path "/78e1f998-c6c8-4383-a798-619907ba92a3"
 					(reference "#PWR02")
@@
 		)
 		(instances
-			(project "barrel-roll"
+			(project "barrel-roll-DIPPCB_pro"
 				(path "/78e1f998-c6c8-4383-a798-619907ba92a3"
 					(reference "#PWR08")
@@
 		)
 		(instances
-			(project "barrel-roll"
+			(project "barrel-roll-DIPPCB_pro"
 				(path "/78e1f998-c6c8-4383-a798-619907ba92a3"
 					(reference "#PWR01")
@@
 		)
 		(instances
-			(project "barrel-roll"
+			(project "barrel-roll-DIPPCB_pro"
 				(path "/78e1f998-c6c8-4383-a798-619907ba92a3"
 					(reference "U3")
@@
 		)
 		(instances
-			(project "barrel-roll"
+			(project "barrel-roll-DIPPCB_pro"
 				(path "/78e1f998-c6c8-4383-a798-619907ba92a3"
 					(reference "#PWR09")
@@
 		)
 		(instances
-			(project "barrel-roll"
+			(project "barrel-roll-DIPPCB_pro"
 				(path "/78e1f998-c6c8-4383-a798-619907ba92a3"
 					(reference "#PWR04")
@@
 		)
 		(instances
-			(project "barrel-roll"
+			(project "barrel-roll-DIPPCB_pro"
 				(path "/78e1f998-c6c8-4383-a798-619907ba92a3"
 					(reference "#PWR05")
@@
 		)
 		(instances
-			(project "barrel-roll"
+			(project "barrel-roll-DIPPCB_pro"
 				(path "/78e1f998-c6c8-4383-a798-619907ba92a3"
 					(reference "#PWR07")
@@
 		)
 		(instances
-			(project "barrel-roll"
+			(project "barrel-roll-DIPPCB_pro"
 				(path "/78e1f998-c6c8-4383-a798-619907ba92a3"
 					(reference "M1")
@@
 		)
 		(instances
-			(project "barrel-roll"
+			(project "barrel-roll-DIPPCB_pro"
 				(path "/78e1f998-c6c8-4383-a798-619907ba92a3"
 					(reference "TP3")
@@
 			)
 		)
-		(property "Footprint" "Seeed Studio XIAO Series Library:XIAO-RP2040-SMD"
+		(property "Footprint" "Seeed Studio XIAO Series Library:XIAO-RP2040-DIP"
 			(at 123.698 117.348 0)
 			(hide yes)
@@
 		)
 		(instances
-			(project "barrel-roll"
+			(project "barrel-roll-DIPPCB_pro"
 				(path "/78e1f998-c6c8-4383-a798-619907ba92a3"
 					(reference "U1")
@@
 		)
 		(instances
-			(project "barrel-roll"
+			(project "barrel-roll-DIPPCB_pro"
 				(path "/78e1f998-c6c8-4383-a798-619907ba92a3"
 					(reference "#PWR06")
@@
 		)
 		(instances
-			(project "barrel-roll"
+			(project "barrel-roll-DIPPCB_pro"
 				(path "/78e1f998-c6c8-4383-a798-619907ba92a3"
 					(reference "TP4")
@@
 		)
 		(instances
-			(project "barrel-roll"
+			(project "barrel-roll-DIPPCB_pro"
 				(path "/78e1f998-c6c8-4383-a798-619907ba92a3"
 					(reference "U2")
@@
 		)
 		(instances
-			(project "barrel-roll"
+			(project "barrel-roll-DIPPCB_pro"
 				(path "/78e1f998-c6c8-4383-a798-619907ba92a3"
 					(reference "XT1")
