File: Electronics/barrel-roll-pcb/barrel-roll.kicad_sch (KiCad schematic)
At the start: 11 parts, among them M1 Motor_DC, M2 Motor_DC, U1 XIAO-RP2040-DIP, U2 DRV8833PW, U3 WeaponMotor, U4 Recever

Commit message: WOrked on the assembly instructions
horrible progress
Other:
- title: (none) -> Barrel Roll Schematic
Changed lines of the file:
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@@
 	(generator_version "10.0")
 	(paper "A4")
+	(title_block
+		(title "Barrel Roll Schematic")
+		(rev "0")
+	)
 	(wire
 		(pts
